File: ELI2350Dock/ELI2350Dock.kicad_pcb (KiCad board)
At the start: 4 copper layers, 219 x 50.7 mm, 13 parts, among them J1 Conn_01x32_Pin, J2 Conn_01x32_Pin

Commit message: doc pre-reroute
Parts:
- CN2: footprint emutelab:CONN-SMD_HC-PBB23L-60DP-0.5V8-G2-01 -> emutelab:CONN-SMD_HC-PBB23L-60DP-0.5V10-G2-01
Routing:
- net +12V: track 263.6 -> 0.00 mm, vias 5 -> 0
- net /~{BOOTSEL}: track 249.6 -> 0.00 mm, vias 1 -> 0
- net /+3V3_SIG: track 241.2 -> 0.00 mm, vias 2 -> 0
- net /GPIO16: track 233.6 -> 0.00 mm, vias 3 -> 0
- net /GPIO23: track 207.8 -> 0.00 mm, vias 5 -> 0
- net /GPIO15: track 206.5 -> 0.00 mm, vias 4 -> 0
- net /GPIO39: track 206.2 -> 0.00 mm, vias 4 -> 0
- net /GPIO9: track 205.0 -> 0.00 mm, vias 5 -> 0
- net /GPIO37: track 204.9 -> 0.00 mm, vias 5 -> 0
- net /GPIO27: track 203.3 -> 0.00 mm, vias 5 -> 0
- net /GPIO36: track 201.9 -> 0.00 mm, vias 4 -> 0
- net /GPIO1: track 200.3 -> 0.00 mm, vias 3 -> 0
- net /GPIO7: track 199.5 -> 0.00 mm, vias 5 -> 0
- net /GPIO29: track 198.7 -> 0.00 mm, vias 5 -> 0
- net /GPIO26: track 197.9 -> 0.00 mm, vias 5 -> 0
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
Commit message: bboard
Parts:
- removed C7, C9: 22u, Capacitor_SMD:C_0805_2012Metric
- added C1: 22u El, Capacitor_SMD:CP_Elec_4x3.9, F.Cu at (124.6, 60.6)
- added C2: 22u El, Capacitor_SMD:CP_Elec_4x3.9, F.Cu at (116.7, 53.4)
- moved C13 10.1 mm to (133.5, 60.0)
- moved C19 10.0 mm to (123.0, 48.9)
- moved D2 8.31 mm to (127.5, 48.9), turned to 180 degrees
- moved FB1 4.14 mm to (132.1, 48.9), turned to 180 degrees
- moved FB2 3.20 mm to (131.3, 53.4), turned to 180 degrees
Connections:
- CN2 pad 1: +12V -> /USB_D_CX+
- CN2 pad 10: /GPIO3 -> /GPIO14
- CN2 pad 11: /GPIO4 -> /GPIO13
- CN2 pad 12: /GPIO5 -> /GPIO12
- CN2 pad 13: /GPIO6 -> /GPIO11
- CN2 pad 14: /GPIO7 -> /GPIO10
- CN2 pad 15: /GPIO8 -> /GPIO9
- CN2 pad 16: /GPIO9 -> /GPIO8
- CN2 pad 17: /GPIO10 -> /GPIO7
- CN2 pad 18: /GPIO11 -> /GPIO6
- CN2 pad 19: /GPIO12 -> /GPIO5
- CN2 pad 2: +5V -> /USB_D_CX-
- CN2 pad 20: /GPIO13 -> /GPIO4
- CN2 pad 21: /GPIO14 -> /GPIO3
- CN2 pad 22: /GPIO15 -> /GPIO2
- CN2 pad 23: /GPIO16 -> /GPIO1
- CN2 pad 24: /GPIO17 -> /GPIO0
- CN2 pad 25: /GPIO18 -> GND
- CN2 pad 26: /GPIO19 -> /+3V3_SIG
- CN2 pad 27: /GPIO20 -> GND
- CN2 pad 28: GND -> +3V3
- CN2 pad 29: /USB_D_CX- -> +5V
- CN2 pad 3: +3V3 -> GND
- CN2 pad 30: /USB_D_CX+ -> +12V
- CN2 pad 31: /~{RESET} -> /GPIO47
- CN2 pad 32: /~{BOOTSEL} -> /GPIO46
- CN2 pad 33: /GPIO21 -> /GPIO45
- CN2 pad 34: /GPIO22 -> /GPIO44
- CN2 pad 35: /GPIO23 -> /GPIO43
- CN2 pad 36: /GPIO24 -> /GPIO42
- CN2 pad 37: /GPIO25 -> /GPIO41
- CN2 pad 38: /GPIO26 -> /GPIO40
- CN2 pad 39: /GPIO27 -> GND
- CN2 pad 4: GND -> /GPIO20
- CN2 pad 40: /GPIO28 -> /GPIO39
- CN2 pad 41: /GPIO29 -> /GPIO38
- CN2 pad 42: /GPIO30 -> /GPIO37
- CN2 pad 43: /GPIO31 -> /GPIO36
- CN2 pad 44: /GPIO32 -> /GPIO35
- CN2 pad 45: /GPIO33 -> /GPIO34
- CN2 pad 46: /GPIO34 -> /GPIO33
- CN2 pad 47: /GPIO35 -> /GPIO32
- CN2 pad 48: /GPIO36 -> /GPIO31
- CN2 pad 49: /GPIO37 -> /GPIO30
- CN2 pad 5: /+3V3_SIG -> /GPIO19
- CN2 pad 50: /GPIO38 -> /GPIO29
- CN2 pad 51: /GPIO39 -> /GPIO28
- CN2 pad 52: GND -> /GPIO27
- CN2 pad 53: /GPIO40 -> /GPIO26
- CN2 pad 54: /GPIO41 -> /GPIO25
- CN2 pad 55: /GPIO42 -> /GPIO24
- CN2 pad 56: /GPIO43 -> /GPIO23
- CN2 pad 57: /GPIO44 -> /GPIO22
- CN2 pad 58: /GPIO45 -> /GPIO21
- CN2 pad 59: /GPIO46 -> /~{BOOTSEL}
- CN2 pad 6: GND -> /GPIO18
- CN2 pad 60: /GPIO47 -> /~{RESET}
- CN2 pad 7: /GPIO0 -> /GPIO17
- CN2 pad 8: /GPIO1 -> /GPIO16
- CN2 pad 9: /GPIO2 -> /GPIO15
Routing:
- net /GPIO8: track 0.00 -> 232.9 mm, vias 0 -> 2
- net /~{BOOTSEL}: track 0.00 -> 232.1 mm, vias 0 -> 1
- net +12V: track 0.00 -> 219.6 mm, vias 0 -> 4
- net /GPIO28: track 0.00 -> 213.3 mm, vias 0 -> 5
- net /GPIO19: track 0.00 -> 208.5 mm, vias 0 -> 3
- net /GPIO22: track 0.00 -> 207.9 mm, vias 0 -> 3
- net /GPIO33: track 0.00 -> 207.5 mm, vias 0 -> 5
- net /~{RESET}: track 0.00 -> 205.7 mm, vias 0 -> 2
- net /GPIO13: track 0.00 -> 205.0 mm, vias 0 -> 4
- net /GPIO21: track 0.00 -> 203.7 mm, vias 0 -> 2
- net /GPIO27: track 0.00 -> 202.4 mm, vias 0 -> 4
- net /GPIO10: track 0.00 -> 202.3 mm, vias 0 -> 3
- net /GPIO20: track 0.00 -> 201.6 mm, vias 0 -> 1
- net /GPIO15: track 0.00 -> 200.8 mm, vias 0 -> 5
- net /GPIO32: track 0.00 -> 200.6 mm, vias 0 -> 3
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Other:
- board text added: "Emute Lab Instruments ELI2350 Dock v0.2 December 2025"
- board text removed: "Emute Lab Instruments ELI2350 Dock v0.1 November 2025"
